File: _saved_hvac.sch (KiCad schematic (older format))
At the start: 44 parts, among them IC1 ATMEGA328P-A, J1 PROGRAMMING HEADER, J2 SERIAL PORT, J3 POWER_INPUT, M1 PINHD-1X10, SW1 SPST, SW2 SPST, SW3 SPST, U1 MIC5225, U2 MOSFET_N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

Commit message: Add some footprints
Parts:
- removed M1: PINHD-1X10, Air_Coils_SML_NEOSID:Neosid_Air-Coil_SML_1turn_HDM0131A, symbol PINHD-1X10
- added JP2: PINHD-1X9, homebrew:1x9-0534260910, symbol PINHD-1X9
- BTN1: footprint (none) -> homebrew:EG2355-ND
- F1: footprint Air_Coils_SML_NEOSID:Neosid_Air-Coil_SML_1turn_HDM0131A -> homebrew:FUSE-3550-2
- RV1, RV2: footprint Air_Coils_SML_NEOSID:Neosid_Air-Coil_SML_1turn_HDM0131A -> homebrew:PDB12-H4301-103BF
- SW1, SW2, SW3: footprint Air_Coils_SML_NEOSID:Neosid_Air-Coil_SML_1turn_HDM0131A -> homebrew:EG2355-ND
Connections:
- net AUX: now also JP2.9
- net GND: now also JP2.3, JP2.6, JP2.8
- net SW_WATER_LIMIT: now also JP2.7
- net TEMP_INSIDE: now also JP2.1
- net TEMP_OUTSIDE: now also JP2.4
- net VCC: now also JP2.2, JP2.5
Changed lines of the file:
@@
 F 0 "SW1" H 9500 800 50  0000 C CNN
 F 1 "SPST" H 9500 600 50  0000 C CNN
-F 2 "Air_Coils_SML_NEOSID:Neosid_Air-Coil_SML_1turn_HDM0131A" H 9500 700 50  0001 C CNN
+F 2 "homebrew:EG2355-ND" H 9500 700 50  0001 C CNN
 F 3 "" H 9500 700 50  0000 C CNN
 	1    9500 700
@@
 F 0 "SW2" H 9500 1050 50  0000 C CNN
 F 1 "SPST" H 9500 850 50  0000 C CNN
-F 2 "Air_Coils_SML_NEOSID:Neosid_Air-Coil_SML_1turn_HDM0131A" H 9500 950 50  0001 C CNN
+F 2 "homebrew:EG2355-ND" H 9500 950 50  0001 C CNN
 F 3 "" H 9500 950 50  0000 C CNN
 	1    9500 950
@@
 F 0 "SW3" H 9500 1300 50  0000 C CNN
 F 1 "SPST" H 9500 1100 50  0000 C CNN
-F 2 "Air_Coils_SML_NEOSID:Neosid_Air-Coil_SML_1turn_HDM0131A" H 9500 1200 50  0001 C CNN
+F 2 "homebrew:EG2355-ND" H 9500 1200 50  0001 C CNN
 F 3 "" H 9500 1200 50  0000 C CNN
 	1    9500 1200
@@
 F 0 "RV1" H 9350 1920 50  0000 C CNN
 F 1 "POT" H 9350 2000 50  0000 C CNN
-F 2 "Air_Coils_SML_NEOSID:Neosid_Air-Coil_SML_1turn_HDM0131A" H 9350 2000 50  0001 C CNN
+F 2 "homebrew:PDB12-H4301-103BF" H 9350 2000 50  0001 C CNN
 F 3 "" H 9350 2000 50  0000 C CNN
 	1    9350 2000
@@
 F 0 "RV2" H 9350 2470 50  0000 C CNN
 F 1 "POT" H 9350 2550 50  0000 C CNN
-F 2 "Air_Coils_SML_NEOSID:Neosid_Air-Coil_SML_1turn_HDM0131A" H 9350 2550 50  0001 C CNN
+F 2 "homebrew:PDB12-H4301-103BF" H 9350 2550 50  0001 C CNN
 F 3 "" H 9350 2550 50  0000 C CNN
 	1    9350 2550
@@
 F 0 "BTN1" H 9500 1550 50  0000 C CNN
 F 1 "SPST" H 9500 1350 50  0001 C CNN
-F 2 "" H 9500 1450 50  0001 C CNN
+F 2 "homebrew:EG2355-ND" H 9500 1450 50  0001 C CNN
 F 3 "" H 9500 1450 50  0000 C CNN
 	1    9500 1450
@@
 F 0 "F1" H 3800 6150 50  0000 L BNN
 F 1 "POWER_FUSE" H 4400 6150 50  0000 L BNN
-F 2 "Air_Coils_SML_NEOSID:Neosid_Air-Coil_SML_1turn_HDM0131A" H 4230 6200 20  0001 C CNN
+F 2 "homebrew:FUSE-3550-2" H 4230 6200 20  0001 C CNN
 F 3 "" H 4200 6050 60  0000 C CNN
 	1    4200 6050
@@
 Text Notes 350  6400 0    60   ~ 0
 TODO: Verify programming port
-$Comp
-L PINHD-1X10 M1
-U 1 1 5910F906
-P 10450 3650
-F 0 "M1" H 10200 4175 50  0000 L BNN
-F 1 "PINHD-1X10" H 10200 2950 50  0000 L BNN
-F 2 "Air_Coils_SML_NEOSID:Neosid_Air-Coil_SML_1turn_HDM0131A" H 10480 3800 20  0001 C CNN
-F 3 "" H 10450 3650 60  0000 C CNN
-	1    10450 3650
-	1    0    0    -1
-$EndComp
 Wire Wire Line
 	9150 3200 9150 3650
@@
 	10350 3950 9250 3950
 Connection ~ 9250 3950
-Wire Wire Line
-	9250 4150 10350 4150
 Connection ~ 9250 4150
 Wire Wire Line
@@
 Wire Wire Line
 	1200 1500 1950 1500
+$Comp
+L PINHD-1X9 JP2
+U 1 1 591172FD
+P 10450 3650
+F 0 "JP2" H 10200 4175 50  0000 L BNN
+F 1 "PINHD-1X9" H 10200 3050 50  0000 L BNN
+F 2 "homebrew:1x9-0534260910" H 10480 3800 20  0001 C CNN
+F 3 "" H 10450 3650 60  0000 C CNN
+	1    10450 3650
+	1    0    0    -1
+$EndComp
 $EndSCHEMATC
