File: hvac.kicad_pcb (KiCad board)
At the start: 2 copper layers, 191.8 x 114.3 mm, 44 parts, among them IC1 ATMEGA328P-A, J1 PROGRAMMING HEADER, J2 SERIAL PORT, J3 POWER_INPUT, SW1 SPST, SW2 SPST, SW3 SPST, U1 MIC5225, U2 MOSFET_N, U3 MOSFET_N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

Commit message: Lay out all the parts in semi logical places
Parts:
- moved C1 99.0 mm to (206.8, 145.0)
- moved R11 96.1 mm to (201.0, 96.0)
- moved R14 93.2 mm to (201.0, 94.5)
- moved R15 84.1 mm to (201.0, 99.6), turned to 180 degrees
- moved R12 83.9 mm to (201.0, 98.0), turned to 180 degrees
- moved R4 81.6 mm to (188.0, 127.0), turned to 270 degrees
- moved C3 80.2 mm to (179.0, 135.0)
- moved SW3 76.8 mm to (171.0, 63.0), turned to 90 degrees
- moved R10 65.4 mm to (201.0, 91.0)
- moved C2 64.6 mm to (179.0, 120.0)
- moved R1 62.7 mm to (217.4, 105.0)
- moved SW2 59.2 mm to (171.0, 79.6), turned to 270 degrees
- moved R2 56.7 mm to (215.0, 105.0)
- moved RV2 51.1 mm to (199.0, 63.0), turned to 90 degrees
- moved R16 47.0 mm to (203.0, 58.5), turned to 90 degrees
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