File: hvac.kicad_pcb (KiCad board)
At the start: 2 copper layers, 76.5 x 99 mm, 51 parts, among them IC1 ATMEGA328P-A, J1 PROGRAMMING HEADER, J2 SERIAL PORT, J3 POWER_INPUT, M1 FIDUCIAL, M2 FIDUCIAL, M3 FIDUCIAL, SW1 SPST, SW2 SPST, SW3 SPST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

Commit message: Add pullup resistors for temperature probes
Parts:
- added R18: 4.7k, Resistors_SMD:R_0402, F.Cu at (61.0, 122.0)
- added R19: 4.7k, Resistors_SMD:R_0402, F.Cu at (65.5, 120.5)
Routing:
- net VCC: track 136.6 -> 145.7 mm
- net GND: track 227.0 -> 235.3 mm
- net TEMP_OUTSIDE: track 22.7 -> 25.2 mm
- net TEMP_INSIDE: track 23.7 -> 25.0 mm
- net OUT_PUMP: track 102.6 -> 103.5 mm
Changed lines of the file:
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@@
 (kicad_pcb (version 4) (host pcbnew 4.0.2+dfsg1-stable)
   (general
-    (links 253)
-    (no_connects 10)
-    (area 47.753858 36.924999 126.075001 136.075001)
+    (links 257)
+    (no_connects 7)
+    (area 47.753858 36.924999 128.175001 136.075001)
     (thickness 1.6)
     (drawings 20)
-    (tracks 700)
+    (tracks 720)
     (zones 0)
-    (modules 51)
+    (modules 53)
     (nets 46)
   )
@@
   (layers
     (0 F.Cu signal)
-    (31 B.Cu signal hide)
+    (31 B.Cu signal)
     (32 B.Adhes user)
     (33 F.Adhes user)
@@
   )
   (setup
-    (last_trace_width 5)
+    (last_trace_width 0.5)
     (user_trace_width 0.5)
     (user_trace_width 1)
@@
       (net 20 SW_SWAMP))
   )
+  (module Resistors_SMD:R_0402 (layer F.Cu)
+    (at 61.05 122)
+    (descr "Resistor SMD 0402, reflow soldering, Vishay (see dcrcw.pdf)")
+    (tags "resistor 0402")
+    (attr smd)
+    (fp_text reference R18 (at 0 -1.8) (layer F.SilkS)
+      (effects (font (size 1 1) (thickness 0.15)))
+    )
+    (fp_text value 4.7k (at 0 1.8) (layer F.Fab)
+      (effects (font (size 1 1) (thickness 0.15)))
+    )
+    (fp_line (start -0.95 -0.65) (end 0.95 -0.65) (layer F.CrtYd) (width 0.05))
+    (fp_line (start -0.95 0.65) (end 0.95 0.65) (layer F.CrtYd) (width 0.05))
+    (fp_line (start -0.95 -0.65) (end -0.95 0.65) (layer F.CrtYd) (width 0.05))
+    (fp_line (start 0.95 -0.65) (end 0.95 0.65) (layer F.CrtYd) (width 0.05))
+    (fp_line (start 0.25 -0.525) (end -0.25 -0.525) (layer F.SilkS) (width 0.15))
+    (fp_line (start -0.25 0.525) (end 0.25 0.525) (layer F.SilkS) (width 0.15))
+    (pad 1 smd rect (at -0.45 0) (size 0.4 0.6) (layers F.Cu F.Paste F.Mask)
+      (net 5 VCC))
+    (pad 2 smd rect (at 0.45 0) (size 0.4 0.6) (layers F.Cu F.Paste F.Mask)
+      (net 15 TEMP_OUTSIDE))
+    (model Resistors_SMD.3dshapes/R_0402.wrl
+      (at (xyz 0 0 0))
+      (scale (xyz 1 1 1))
+      (rotate (xyz 0 0 0))
+    )
+  )
+  (module Resistors_SMD:R_0402 (layer F.Cu)
+    (at 65.5 120.5 180)
+    (descr "Resistor SMD 0402, reflow soldering, Vishay (see dcrcw.pdf)")
+    (tags "resistor 0402")
+    (attr smd)
+    (fp_text reference R19 (at 0 -1.8 180) (layer F.SilkS)
+      (effects (font (size 1 1) (thickness 0.15)))
+    )
+    (fp_text value 4.7k (at 0 1.8 180) (layer F.Fab)
+      (effects (font (size 1 1) (thickness 0.15)))
+    )
+    (fp_line (start -0.95 -0.65) (end 0.95 -0.65) (layer F.CrtYd) (width 0.05))
+    (fp_line (start -0.95 0.65) (end 0.95 0.65) (layer F.CrtYd) (width 0.05))
+    (fp_line (start -0.95 -0.65) (end -0.95 0.65) (layer F.CrtYd) (width 0.05))
+    (fp_line (start 0.95 -0.65) (end 0.95 0.65) (layer F.CrtYd) (width 0.05))
+    (fp_line (start 0.25 -0.525) (end -0.25 -0.525) (layer F.SilkS) (width 0.15))
+    (fp_line (start -0.25 0.525) (end 0.25 0.525) (layer F.SilkS) (width 0.15))
+    (pad 1 smd rect (at -0.45 0 180) (size 0.4 0.6) (layers F.Cu F.Paste F.Mask)
+      (net 5 VCC))
+    (pad 2 smd rect (at 0.45 0 180) (size 0.4 0.6) (layers F.Cu F.Paste F.Mask)
+      (net 16 TEMP_INSIDE))
+    (model Resistors_SMD.3dshapes/R_0402.wrl
+      (at (xyz 0 0 0))
+      (scale (xyz 1 1 1))
+      (rotate (xyz 0 0 0))
+    )
+  )
   (gr_text RST (at 52 93.5) (layer F.SilkS)
     (effects (font (size 1.5 1.5) (thickness 0.3)))
@@
   (gr_line (start 126 37) (end 126 136) (angle 90) (layer Edge.Cuts) (width 0.15))
   (gr_line (start 49.5 37) (end 125.97 37) (angle 90) (layer Edge.Cuts) (width 0.15))
+  (segment (start 88.5014 48) (end 88.5014 48.89878) (width 0.5) (layer F.Cu) (net 1))
+  (segment (start 88.5014 48.89878) (end 90.79762 51.195) (width 0.5) (layer F.Cu) (net 1))
+  (segment (start 90.79762 51.195) (end 91.3 51.195) (width 0.5) (layer F.Cu) (net 1))
+  (segment (start 55.3 85.2) (end 53.744366 85.2) (width 0.5) (layer B.Cu) (net 1))
+  (segment (start 53.744366 85.2) (end 53.444366 85.5) (width 0.5) (layer B.Cu) (net 1))
+  (segment (start 55.3 90.78) (end 56.239799 89.840201) (width 0.5) (layer B.Cu) (net 1))
+  (segment (start 56.239799 89.840201) (end 56.659799 89.840201) (width 0.5) (layer B.Cu) (net 1))
   (segment (start 88.5014 48) (end 88.5014 41.9014) (width 0.5) (layer F.Cu) (net 1))
   (segment (start 88.5014 41.9014) (end 88.1 41.5) (width 0.5) (layer F.Cu) (net 1))
@@
   (segment (start 67.7 97.3) (end 67.7 97.4) (width 0.5) (layer F.Cu) (net 4))
   (segment (start 67.70234 97.40234) (end 67.7 97.4) (width 0.5) (layer F.Cu) (net 4))
+  (segment (start 65.95 120.5) (end 65.95 122.85) (width 0.5) (layer F.Cu) (net 5))
+  (segment (start 65.95 122.85) (end 69.3 126.2) (width 0.5) (layer F.Cu) (net 5))
+  (segment (start 60.6 122) (end 60.6 125) (width 0.5) (layer F.Cu) (net 5))
+  (segment (start 60.6 125) (end 61.8 126.2) (width 0.5) (layer F.Cu) (net 5))
+  (segment (start 65.95 120.5) (end 65.95 120.6) (width 0.5) (layer F.Cu) (net 5))
   (segment (start 83.5 73) (end 83.5 70.6) (width 0.5) (layer F.Cu) (net 5))
   (segment (start 83.5 70.6) (end 83.3 70.4) (width 0.5) (layer F.Cu) (net 5))
@@
   (segment (start 61.8 126.2) (end 61.8 127.472792) (width 0.5) (layer F.Cu) (net 5))
   (segment (start 61.8 127.472792) (end 62 127.672792) (width 0.5) (layer F.Cu) (net 5))
-  (segment (start 69.5 124) (end 69.5 123.5) (width 0.5) (layer F.Cu) (net 5))
-  (segment (start 69.3 124.2) (end 69.5 124) (width 0.5) (layer F.Cu) (net 5))
-  (segment (start 69.3 126.2) (end 69.3 124.2) (width 0.5) (layer F.Cu) (net 5))
   (segment (start 71 96) (end 71 95.5) (width 0.5) (layer F.Cu) (net 5))
   (segment (start 86 125.5) (end 86.5 126) (width 0.5) (layer F.Cu) (net 5))
@@
   (segment (start 95.275 112.5) (end 95.3 112.5) (width 0.5) (layer F.Cu) (net 5))
   (segment (start 95.166 112.366) (end 95.3 112.5) (width 0.25) (layer F.Cu) (net 5))
-  (segment (start 117.3 82.5) (end 117.3 92.5) (width 5) (layer F.Cu) (net 6))
+  (segment (start 117.3 82.5) (end 117.3 87.5) (width 5) (layer F.Cu) (net 6))
+  (segment (start 117.3 87.5) (end 117.3 92.5) (width 5) (layer F.Cu) (net 6))
+  (segment (start 117.3 87.4) (end 117.3 87.5) (width 0.5) (layer F.Cu) (net 6))
   (segment (start 117.3 92.5) (end 121.3 96.5) (width 5) (layer F.Cu) (net 6))
   (segment (start 98.356001 100.556001) (end 117.243999 100.556001) (width 5) (layer B.Cu) (net 6))
@@
   (segment (start 62.50842 102.20842) (end 62.5 102.2) (width 0.5) (layer F.Cu) (net 14))
   (via (at 62.5 102.2) (size 0.6) (drill 0.4) (layers F.Cu B.Cu) (net 14))
+  (segment (start 62.723519 106.367079) (end 62.723519 120.5) (width 0.5) (layer F.Cu) (net 15))
+  (segment (start 62.723519 120.5) (end 62.723519 121) (width 0.5) (layer F.Cu) (net 15))
+  (segment (start 61.5 122) (end 61.5 121.9) (width 0.5) (layer F.Cu) (net 15))
+  (segment (start 62.723519 120.676481) (end 62.723519 120.5) (width 0.5) (layer F.Cu) (net 15))
+  (segment (start 61.5 121.9) (end 62.723519 120.676481) (width 0.5) (layer F.Cu) (net 15))
+  (segment (start 62.723519 121) (end 62.723519 122.123519) (width 0.5) (layer F.Cu) (net 15))
+  (segment (start 62.723519 121.476481) (end 62.723519 121) (width 0.5) (layer F.Cu) (net 15))
   (segment (start 63.80852 106.20638) (end 62.884218 106.20638) (width 0.5) (layer F.Cu) (net 15))
   (segment (start 62.884218 106.20638) (end 62.723519 106.367079) (width 0.5) (layer F.Cu) (net 15))
-  (segment (start 62.723519 106.367079) (end 62.723519 122.123519) (width 0.5) (layer F.Cu) (net 15))
   (segment (start 62.723519 122.123519) (end 65.900001 125.300001) (width 0.5) (layer F.Cu) (net 15))
   (segment (start 65.900001 125.300001) (end 66.8 126.2) (width 0.5) (layer F.Cu) (net 15))
+  (segment (start 65.05 120.5) (end 63.9 120.5) (width 0.5) (layer F.Cu) (net 16))
+  (segment (start 63.9 120.5) (end 63.8 120.6) (width 0.5) (layer F.Cu) (net 16))
   (segment (start 59.3 120.6) (end 59.3 126.2) (width 0.5) (layer F.Cu) (net 16))
   (segment (start 63.8 120.6) (end 59.3 120.6) (width 0.5) (layer B.Cu) (net 16))
@@
   (segment (start 65.30204 97.40204) (end 65.3 97.4) (width 0.5) (layer F.Cu) (net 35))
   (via (at 65.3 97.4) (size 0.6) (drill 0.4) (layers F.Cu B.Cu) (net 35))
+  (segment (start 101.1 48.75) (end 101.1 49.65) (width 0.5) (layer B.Cu) (net 36))
   (segment (start 106.144 52.524) (end 109.344 52.524) (width 0.5) (layer F.Cu) (net 36))
   (segment (start 96.6 49.65) (end 96.6 51.35) (width 0.5) (layer B.Cu) (net 36))

Commit message: Bump revision + minor changes
Parts:
- R8: value 2.2k -> 3.3k
Other:
- board text added: "+"
- board text added: "-"
- board text added: "HVAC V1.1"
- board text removed: "HVAC V1.0"
Changed lines of the file:
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@@
     (area 47.753858 36.924999 128.175001 136.075001)
     (thickness 1.6)
-    (drawings 20)
+    (drawings 22)
     (tracks 720)
     (zones 0)
@@
       (effects (font (size 1 1) (thickness 0.15)))
     )
-    (fp_text value 2.2k (at 0 1.8 180) (layer F.Fab)
+    (fp_text value 3.3k (at 0 1.8 180) (layer F.Fab)
       (effects (font (size 1 1) (thickness 0.15)))
     )
@@
     )
   )
+  (gr_text - (at 105.5 117) (layer F.SilkS)
+    (effects (font (size 4 4) (thickness 0.3)))
+  )
+  (gr_text + (at 105.5 131) (layer F.SilkS)
+    (effects (font (size 4 4) (thickness 0.3)))
+  )
   (gr_text RST (at 52 93.5) (layer F.SilkS)
     (effects (font (size 1.5 1.5) (thickness 0.3)))
@@
   (gr_line (start 54 106) (end 54 108) (layer F.SilkS) (width 0.2))
   (gr_line (start 53 106) (end 54 106) (layer F.SilkS) (width 0.2))
-  (gr_text "HVAC V1.0" (at 56 112 270) (layer F.SilkS)
+  (gr_text "HVAC V1.1" (at 56 112 270) (layer F.SilkS)
     (effects (font (size 1.5 1.5) (thickness 0.3)))
   )
